File: nab.kicad_pcb (KiCad board)
At the start: 2 copper layers, 20 x 110 mm, 21 parts, among them J1 MIX LINE OUT, J2 LINE IN, J3 LINE OUT, J4 MOD IN L, J5 MOD IN R, J6 Conn_01x03_Male, J7 Conn_01x03_Male, J8 Conn_01x03_Male, J9 Conn_01x03_Male

Commit message: rev2 (missed a ground)
Connections:
- J3 pad S: Net-(J3-PadS) -> GND
Other:
- board text added: "REV2"
