File: nab.sch (KiCad schematic (older format))
At the start: 19 parts, among them J1 MIX LINE OUT, J2 LINE IN, J3 LINE OUT, J4 MOD IN L, J5 MOD IN R, J6 Conn_01x03_Male, J7 Conn_01x03_Male, J8 Conn_01x03_Male, J9 Conn_01x03_Male

Commit message: rev2 (missed a ground)
Connections:
- net GND: now also J3.S
Changed lines of the file:
@@
 Wire Wire Line
 	6300 4300 6550 4300
+$Comp
+L power:GND #PWR?
+U 1 1 5FC875BC
+P 2750 1300
+F 0 "#PWR?" H 2750 1050 50  0001 C CNN
+F 1 "GND" H 2755 1127 50  0000 C CNN
+F 2 "" H 2750 1300 50  0001 C CNN
+F 3 "" H 2750 1300 50  0001 C CNN
+	1    2750 1300
+	1    0    0    -1
+$EndComp
+Wire Wire Line
+	2350 1500 2350 1300
+Wire Wire Line
+	2350 1300 2750 1300
 $EndSCHEMATC

Commit message: rev2
Other:
- note removed: "NOTES:\n\nCan make it Intellijel 1u wide/highX eurorack height: 39.65mm X 128.5mm\n\nAlthough, it’s about 8hp, which is large, might be better to just to a 1u tile size PCB with 2x panels, one for 1U and one for == to the internal PCB dims?"
Changed lines of the file:
@@
 Text Notes 9300 1700 0    50   ~ 0
 Line OUT R
-Text Notes 3250 1050 0    50   ~ 0
-NOTES:\n\nCan make it Intellijel 1u wide/highX eurorack height:   39.65mm X 128.5mm\n\nAlthough, it’s about 8hp, which is large, might be better to just to a 1u tile size PCB with 2x panels, one for 1U and one for == to the internal PCB dims?
 $Comp
 L thonkiconn_symbol:thonkiconn J5
